Commit message: fix: spatial accuracy corrections from multi-model validation
- AprilTags: vertical orientation (pitch ±π/2) at Z=0.25m (camera height),
  facing robot approach direction, using real tag36h11 textures via PBR
- Heating rails: corrected rotation (pitch π/2 instead of roll π/2) so
  pipes run alongside crop rows (+X axis) instead of across aisles
- Lidar: raised to Z=0.10 (above chassis top at Z=0.075)
- Drive shaping: safe default invert_right=false for simulation
- Markers registry: updated to match corrected tag poses
- AprilTag model SDFs: migrated from Ogre1 scripts to SDF 1.9 PBR materials

Validated by: GPT-5.4, Gemini 3.1 Pro, and mathematical verification.

File: src/agv_sim_description/urdf/sensors_sim.xacro (robot description, xacro)
@@ -215,5 +215,5 @@
     <parent link="base_link"/>
     <child link="laser_frame"/>
-    <origin xyz="0.5 0.0 0.0" rpy="0 0 0"/>
+    <origin xyz="0.5 0.0 0.10" rpy="0 0 0"/>
   </joint>
   <gazebo reference="laser_frame">
