Commit message: refactor: remove fake lidar, use ZED 2i depth-to-laserscan
The real AGV has no lidar — only a ZED 2i stereo camera. Removed
the gpu_lidar sensor and laser_frame from the URDF and the lidar
bridge from gz_bridge.yaml.

Added depthimage_to_laserscan node to sim_external.launch.py which
converts the ZED depth image to /agv/scan (LaserScan). This matches
the standard ZED 2i + Nav2 pattern used by Stereolabs examples.

The scan topic will produce data when depth camera rendering works
(ogre2 GPU sensor pipeline). Same underlying dependency as before,
but now the architecture matches the real robot's sensor suite.

Co-Authored-By: Claude Opus 4.6 (1M context) <noreply@anthropic.com>

File: src/agv_sim_description/urdf/sensors_sim.xacro (robot description, xacro)
@@ -220,67 +220,5 @@
     </sensor>
   </gazebo>
-  <!-- ═══════════════════════════════════════════════════════ -->
-  <!--  2D Lidar (supplementary sensor)                        -->
-  <!-- ═══════════════════════════════════════════════════════ -->
-  <link name="laser_frame">
-    <visual>
-      <geometry>
-        <cylinder radius="0.04" length="0.04"/>
-      </geometry>
-      <material name="lidar_red">
-        <color rgba="0.8 0.0 0.0 1.0"/>
-      </material>
-    </visual>
-    <collision>
-      <geometry>
-        <cylinder radius="0.04" length="0.04"/>
-      </geometry>
-    </collision>
-    <inertial>
-      <mass value="0.1"/>
-      <inertia ixx="0.00005" ixy="0" ixz="0" iyy="0.00005" iyz="0" izz="0.00005"/>
-    </inertial>
-  </link>
-  <joint name="laser_joint" type="fixed">
-    <parent link="base_link"/>
-    <child link="laser_frame"/>
-    <origin xyz="0.5 0.0 0.10" rpy="0 0 0"/>
-  </joint>
-  <gazebo reference="laser_frame">
-    <visual>
-      <material>
-        <ambient>0.6 0.0 0.0 1</ambient>
-        <diffuse>0.8 0.0 0.0 1</diffuse>
-        <specular>0.3 0.1 0.1 1</specular>
-        <pbr><metal><metalness>0.1</metalness><roughness>0.5</roughness></metal></pbr>
-      </material>
-    </visual>
-    <sensor name="lidar_sensor" type="gpu_lidar">
-      <always_on>true</always_on>
-      <visualize>false</visualize>
-      <update_rate>10</update_rate>
-      <topic>/lidar</topic>
-      <gz_frame_id>laser_frame</gz_frame_id>
-      <lidar>
-        <scan>
-          <horizontal>
-            <samples>720</samples>
-            <resolution>1</resolution>
-            <min_angle>-3.14159265359</min_angle>
-            <max_angle>3.14159265359</max_angle>
-          </horizontal>
-        </scan>
-        <range>
-          <min>0.1</min>
-          <max>10.0</max>
-          <resolution>0.01</resolution>
-        </range>
-        <noise>
-          <type>gaussian</type>
-          <mean>0.0</mean>
-          <stddev>0.005</stddev>
-        </noise>
-      </lidar>
-    </sensor>
-  </gazebo>
+  <!-- No lidar — real robot uses ZED 2i depth camera only.
+       /agv/scan is generated by depthimage_to_laserscan from the ZED depth image. -->
 </robot>

Commit message: fix: match real ZED 2i frame names, IMU rate, and camera FPS
Compared against real ZED 2i hardware (S/N 34395516, SDK 5.1.2):

Frame name fixes (match ZED SDK convention):
  zed_left_camera_optical_frame  → zed_left_camera_frame_optical
  zed_right_camera_optical_frame → zed_right_camera_frame_optical

Rate fixes (match real ZED SDK publish rates):
  Camera: 30fps → 15fps (real ZED config: HD1080@15)
  IMU: 400Hz → 100Hz (real ZED config: sensors_publishing_rate=100)

Co-Authored-By: Claude Opus 4.6 (1M context) <noreply@anthropic.com>

File: src/agv_sim_description/urdf/sensors_sim.xacro (robot description, xacro)
@@ -84,13 +84,13 @@
   </joint>
   <!-- Left camera optical frame (rotated for optical convention: Z forward, X right, Y down) -->
-  <link name="zed_left_camera_optical_frame">
-    <inertial>
-      <mass value="0.001"/>
-      <inertia ixx="0.000001" ixy="0" ixz="0" iyy="0.000001" iyz="0" izz="0.000001"/>
-    </inertial>
-  </link>
-  <joint name="zed_left_camera_optical_joint" type="fixed">
+  <link name="zed_left_camera_frame_optical">
+    <inertial>
+      <mass value="0.001"/>
+      <inertia ixx="0.000001" ixy="0" ixz="0" iyy="0.000001" iyz="0" izz="0.000001"/>
+    </inertial>
+  </link>
+  <joint name="zed_left_camera_frame_optical_joint" type="fixed">
     <parent link="zed_left_camera_frame"/>
-    <child link="zed_left_camera_optical_frame"/>
+    <child link="zed_left_camera_frame_optical"/>
     <!-- Rotate -90 deg around Z then -90 deg around X for optical convention -->
     <origin xyz="0 0 0" rpy="${-pi/2} 0 ${-pi/2}"/>
@@ -109,13 +109,13 @@
   </joint>
   <!-- Right camera optical frame -->
-  <link name="zed_right_camera_optical_frame">
-    <inertial>
-      <mass value="0.001"/>
-      <inertia ixx="0.000001" ixy="0" ixz="0" iyy="0.000001" iyz="0" izz="0.000001"/>
-    </inertial>
-  </link>
-  <joint name="zed_right_camera_optical_joint" type="fixed">
+  <link name="zed_right_camera_frame_optical">
+    <inertial>
+      <mass value="0.001"/>
+      <inertia ixx="0.000001" ixy="0" ixz="0" iyy="0.000001" iyz="0" izz="0.000001"/>
+    </inertial>
+  </link>
+  <joint name="zed_right_camera_frame_optical_joint" type="fixed">
     <parent link="zed_right_camera_frame"/>
-    <child link="zed_right_camera_optical_frame"/>
+    <child link="zed_right_camera_frame_optical"/>
     <origin xyz="0 0 0" rpy="${-pi/2} 0 ${-pi/2}"/>
   </joint>
@@ -147,7 +147,7 @@
     <sensor type="depth_camera" name="zed_left_depth">
       <always_on>true</always_on>
-      <update_rate>30</update_rate>
+      <update_rate>15</update_rate>
       <topic>/zed_left</topic>
-      <gz_frame_id>zed_left_camera_optical_frame</gz_frame_id>
+      <gz_frame_id>zed_left_camera_frame_optical</gz_frame_id>
       <camera>
         <horizontal_fov>1.9199</horizontal_fov>
@@ -175,7 +175,7 @@
     <sensor type="camera" name="zed_right_camera">
       <always_on>true</always_on>
-      <update_rate>30</update_rate>
+      <update_rate>15</update_rate>
       <topic>/zed_right</topic>
-      <gz_frame_id>zed_right_camera_optical_frame</gz_frame_id>
+      <gz_frame_id>zed_right_camera_frame_optical</gz_frame_id>
       <camera>
         <horizontal_fov>1.9199</horizontal_fov>
@@ -198,10 +198,10 @@
   </gazebo>
   <!-- ═══════════════════════════════════════════════════════ -->
-  <!--  ZED 2i IMU — 400Hz, datasheet noise values             -->
+  <!--  ZED 2i IMU — 100Hz matching real ZED SDK publish rate   -->
   <!-- ═══════════════════════════════════════════════════════ -->
   <gazebo reference="imu_link">
     <sensor name="zed_imu" type="imu">
       <always_on>true</always_on>
-      <update_rate>400</update_rate>
+      <update_rate>100</update_rate>
       <topic>/zed_imu</topic>
       <gz_frame_id>imu_link</gz_frame_id>
