Commit message: Migrate from Gazebo Classic to Gz Harmonic (Gazebo Sim 8)
Replace gazebo_ros with ros_gz_sim + ros_gz_bridge for Gz Harmonic
compatibility. Key changes:

- World files: .world -> .sdf (SDF 1.9), ODE -> DART physics, inline
  sun light, add Gz system plugins (Physics, Sensors, Imu, etc.)
- URDF plugins: libgazebo_ros_* -> gz-sim-diff-drive-system,
  gz-sim-joint-state-publisher-system; sensors defined natively
  (depth_camera, camera, imu, gpu_lidar) with Gz Transport topics
- Launch files: gazebo_ros gzserver/gzclient -> ros_gz_sim gz_sim,
  spawn_entity.py -> ros_gz_sim create, add ros_gz_bridge nodes
- Bridge config: new gz_bridge.yaml maps all Gz<->ROS topics
  (clock, cmd_vel, odom, cameras, IMU, lidar, joint_states)
- TF control: odom->base_link TF bridged only in teleop/mapping
  modes; omitted in EKF modes (fusion/nav)
- GZ_IP=127.0.0.1 for loopback transport (avoids multicast issues)
- drive_shaping_params: invert_right=false (Gz DiffDrive handles
  wheel direction internally), wildcard node name for namespace match

File: src/agv_sim_description/urdf/agv_base_sim.xacro (robot description, xacro)
@@ -90,17 +90,12 @@
     <origin xyz="-0.25 0 -0.175" rpy="0 0 0"/>
   </joint>
-  <!-- Gazebo friction for casters (low friction to simulate free-rolling) -->
+  <!-- Gz friction for casters (low friction to simulate free-rolling) -->
   <gazebo reference="front_caster">
     <mu1>0.001</mu1>
     <mu2>0.001</mu2>
-    <material>Gazebo/DarkGrey</material>
   </gazebo>
   <gazebo reference="rear_caster">
     <mu1>0.001</mu1>
     <mu2>0.001</mu2>
-    <material>Gazebo/DarkGrey</material>
-  </gazebo>
-  <gazebo reference="base_link">
-    <material>Gazebo/Grey</material>
   </gazebo>
 </robot>

File: src/agv_sim_description/urdf/agv_sim.urdf.xacro (robot description, xacro)
@@ -1,26 +1,23 @@
 <?xml version="1.0"?>
 <!--
-  AGV Simulation Robot Description
+  AGV Simulation Robot Description (Gz Harmonic)
   All dimensions from src/agv_sim_description/config/robot_params.yaml
   Override via xacro args or launch parameters if needed.
   TF chain produced:
     base_link
-      ├── left_wheel     (continuous joint, driven by Gazebo diff_drive)
-      ├── right_wheel    (continuous joint, driven by Gazebo diff_drive)
-      ├── base_footprint (fixed, at ground level)
-      ├── zed_camera_link (fixed, at ZED 2i position)
-      │    ├── zed_camera_center
-      │    ├── zed_left_camera_frame → zed_left_camera_optical_frame
-      │    ├── zed_right_camera_frame → zed_right_camera_optical_frame
-      │    └── imu_link
-      ├── laser_frame    (fixed, front-mounted)
-      ├── front_caster   (fixed, for sim stability)
-      └── rear_caster    (fixed, for sim stability)
-  Gazebo plugins:
-    - libgazebo_ros_diff_drive.so (reads shaped_cmd_vel from drive shaping node)
-    - libgazebo_ros_camera.so (ZED 2i left: RGB + depth + point cloud)
-    - libgazebo_ros_camera.so (ZED 2i right: RGB)
-    - libgazebo_ros_imu_sensor.so (ZED 2i IMU at 400Hz)
-    - libgazebo_ros_ray_sensor.so (2D lidar, supplementary)
+      left_wheel     (continuous joint, driven by Gz DiffDrive)
+      right_wheel    (continuous joint, driven by Gz DiffDrive)
+      base_footprint (fixed, at ground level)
+      zed_camera_link (fixed, at ZED 2i position)
+           zed_camera_center
+           zed_left_camera_frame, zed_right_camera_frame
+           imu_link
+      laser_frame    (fixed, front-mounted)
+      front_caster   (fixed, for sim stability)
+      rear_caster    (fixed, for sim stability)
+  Gz Harmonic plugins:
+    gz sim diff drive system (reads shaped_cmd_vel from drive shaping node)
+    gz sim joint state publisher system (publishes joint states for robot_state_publisher)
+    Sensors: depth_camera, camera, imu, gpu_lidar (bridged to ROS via ros_gz_bridge)
 -->
 <robot xmlns:xacro="http://www.ros.org/wiki/xacro" name="agv">
@@ -31,6 +28,4 @@
   <xacro:arg name="wheel_z"       default="-0.1375"/>
   <xacro:arg name="wheel_width"   default="0.05"/>
-  <!-- Diff drive TF control — set via launch arg for different modes -->
-  <xacro:arg name="publish_odom_tf" default="false"/>
   <!-- Include components -->
   <xacro:include filename="$(find agv_sim_description)/urdf/agv_base_sim.xacro"/>
@@ -54,11 +49,8 @@
     width="$(arg wheel_width)"/>
   <!-- ═══════════════════════════════════════════════════════ -->
-  <!--  Gazebo Diff-Drive Plugin                              -->
+  <!--  Gz Harmonic Diff-Drive Plugin                         -->
   <!-- ═══════════════════════════════════════════════════════ -->
   <gazebo>
-    <plugin name="diff_drive_controller" filename="libgazebo_ros_diff_drive.so">
-      <ros>
-        <remapping>cmd_vel:=cmd_vel</remapping>
-      </ros>
+    <plugin filename="gz-sim-diff-drive-system" name="gz::sim::systems::DiffDrive">
       <!-- Joints -->
       <left_joint>left_wheel_joint</left_joint>
@@ -66,20 +58,22 @@
       <!-- Kinematics -->
       <wheel_separation>0.735</wheel_separation>
-      <wheel_diameter>0.125</wheel_diameter>
-      <!-- Limits -->
-      <max_wheel_torque>20.0</max_wheel_torque>
-      <max_wheel_acceleration>1.0</max_wheel_acceleration>
-      <!-- Odometry output -->
-      <publish_odom>true</publish_odom>
-      <publish_odom_tf>$(arg publish_odom_tf)</publish_odom_tf>
-      <publish_wheel_tf>true</publish_wheel_tf>
+      <wheel_radius>0.0625</wheel_radius>
+      <!-- Topics (Gz Transport — bridged to ROS via ros_gz_bridge) -->
+      <topic>/agv/shaped_cmd_vel</topic>
+      <odom_topic>/agv/wheel_odom</odom_topic>
+      <tf_topic>/agv/tf</tf_topic>
       <!-- Frames -->
-      <odometry_frame>odom</odometry_frame>
-      <robot_base_frame>base_link</robot_base_frame>
-      <!-- Topics -->
-      <command_topic>shaped_cmd_vel</command_topic>
-      <odometry_topic>wheel_odom</odometry_topic>
+      <frame_id>odom</frame_id>
+      <child_frame_id>base_link</child_frame_id>
       <!-- Rate -->
-      <update_rate>50.0</update_rate>
+      <odom_publish_frequency>50</odom_publish_frequency>
+    </plugin>
+  </gazebo>
+  <!-- ═══════════════════════════════════════════════════════ -->
+  <!--  Joint State Publisher (for wheel TF via robot_state_publisher) -->
+  <!-- ═══════════════════════════════════════════════════════ -->
+  <gazebo>
+    <plugin filename="gz-sim-joint-state-publisher-system" name="gz::sim::systems::JointStatePublisher">
+      <topic>/agv/joint_states</topic>
     </plugin>
   </gazebo>

File: src/agv_sim_description/urdf/sensors_sim.xacro (robot description, xacro)
@@ -4,5 +4,5 @@
   <!--  ZED 2i Stereo Camera — TF chain matching real ZED SDK -->
   <!-- ═══════════════════════════════════════════════════════ -->
-  <!-- ZED camera body link (175mm × 30mm × 33mm) -->
+  <!-- ZED camera body link (175mm x 30mm x 33mm) -->
   <link name="zed_camera_link">
     <visual>
@@ -63,5 +63,5 @@
     <parent link="zed_left_camera_frame"/>
     <child link="zed_left_camera_optical_frame"/>
-    <!-- Rotate -90° around Z then -90° around X for optical convention -->
+    <!-- Rotate -90 deg around Z then -90 deg around X for optical convention -->
     <origin xyz="0 0 0" rpy="${-pi/2} 0 ${-pi/2}"/>
   </joint>
@@ -111,10 +111,13 @@
   </joint>
   <!-- ═══════════════════════════════════════════════════════ -->
-  <!--  Left Camera Plugin (RGB + Depth + PointCloud)         -->
+  <!--  Left Camera Sensor (RGB + Depth + PointCloud)          -->
+  <!--  Gz Transport topics bridged to ROS via ros_gz_bridge   -->
   <!-- ═══════════════════════════════════════════════════════ -->
   <gazebo reference="zed_left_camera_frame">
-    <sensor type="depth" name="zed_left_depth">
+    <sensor type="depth_camera" name="zed_left_depth">
       <always_on>true</always_on>
       <update_rate>30</update_rate>
+      <topic>/zed_left</topic>
+      <gz_frame_id>zed_left_camera_optical_frame</gz_frame_id>
       <camera>
         <horizontal_fov>1.9199</horizontal_fov>
@@ -134,22 +137,8 @@
         </noise>
       </camera>
-      <plugin name="zed_left_camera" filename="libgazebo_ros_camera.so">
-        <ros>
-          <namespace>/</namespace>
-          <remapping>image_raw:=zed/zed_node/left/image_rect_color</remapping>
-          <remapping>camera_info:=zed/zed_node/left/camera_info</remapping>
-          <remapping>image_raw/depth:=zed/zed_node/depth/depth_registered</remapping>
-          <remapping>points:=zed/zed_node/point_cloud/cloud_registered</remapping>
-        </ros>
-        <camera_name>zed_left</camera_name>
-        <frame_name>zed_left_camera_optical_frame</frame_name>
-        <hack_baseline>0.12</hack_baseline>
-        <min_depth>0.3</min_depth>
-        <max_depth>20.0</max_depth>
-      </plugin>
-    </sensor>
-  </gazebo>
-  <!-- ═══════════════════════════════════════════════════════ -->
-  <!--  Right Camera Plugin (RGB only)                        -->
+    </sensor>
+  </gazebo>
+  <!-- ═══════════════════════════════════════════════════════ -->
+  <!--  Right Camera Sensor (RGB only)                         -->
   <!-- ═══════════════════════════════════════════════════════ -->
   <gazebo reference="zed_right_camera_frame">
@@ -157,4 +146,6 @@
       <always_on>true</always_on>
       <update_rate>30</update_rate>
+      <topic>/zed_right</topic>
+      <gz_frame_id>zed_right_camera_optical_frame</gz_frame_id>
       <camera>
         <horizontal_fov>1.9199</horizontal_fov>
@@ -174,17 +165,8 @@
         </noise>
       </camera>
-      <plugin name="zed_right_camera" filename="libgazebo_ros_camera.so">
-        <ros>
-          <namespace>/</namespace>
-          <remapping>image_raw:=zed/zed_node/right/image_rect_color</remapping>
-          <remapping>camera_info:=zed/zed_node/right/camera_info</remapping>
-        </ros>
-        <camera_name>zed_right</camera_name>
-        <frame_name>zed_right_camera_optical_frame</frame_name>
-      </plugin>
-    </sensor>
-  </gazebo>
-  <!-- ═══════════════════════════════════════════════════════ -->
-  <!--  ZED 2i IMU — 400Hz, datasheet noise values            -->
+    </sensor>
+  </gazebo>
+  <!-- ═══════════════════════════════════════════════════════ -->
+  <!--  ZED 2i IMU — 400Hz, datasheet noise values             -->
   <!-- ═══════════════════════════════════════════════════════ -->
   <gazebo reference="imu_link">
@@ -192,4 +174,6 @@
       <always_on>true</always_on>
       <update_rate>400</update_rate>
+      <topic>/zed_imu</topic>
+      <gz_frame_id>imu_link</gz_frame_id>
       <imu>
         <angular_velocity>
@@ -204,16 +188,8 @@
         </linear_acceleration>
       </imu>
-      <plugin name="zed_imu_plugin" filename="libgazebo_ros_imu_sensor.so">
-        <ros>
-          <namespace>/</namespace>
-          <remapping>~/out:=zed/zed_node/imu/data</remapping>
-        </ros>
-        <initial_orientation_as_reference>false</initial_orientation_as_reference>
-        <frame_name>imu_link</frame_name>
-      </plugin>
-    </sensor>
-  </gazebo>
-  <!-- ═══════════════════════════════════════════════════════ -->
-  <!--  2D Lidar (supplementary sensor, kept as-is)           -->
+    </sensor>
+  </gazebo>
+  <!-- ═══════════════════════════════════════════════════════ -->
+  <!--  2D Lidar (supplementary sensor)                        -->
   <!-- ═══════════════════════════════════════════════════════ -->
   <link name="laser_frame">
@@ -242,9 +218,11 @@
   </joint>
   <gazebo reference="laser_frame">
-    <sensor name="lidar_sensor" type="ray">
+    <sensor name="lidar_sensor" type="gpu_lidar">
       <always_on>true</always_on>
       <visualize>false</visualize>
       <update_rate>10</update_rate>
-      <ray>
+      <topic>/lidar</topic>
+      <gz_frame_id>laser_frame</gz_frame_id>
+      <lidar>
         <scan>
           <horizontal>
@@ -265,12 +243,5 @@
           <stddev>0.005</stddev>
         </noise>
-      </ray>
-      <plugin name="lidar_plugin" filename="libgazebo_ros_ray_sensor.so">
-        <ros>
-          <remapping>~/out:=scan</remapping>
-        </ros>
-        <output_type>sensor_msgs/LaserScan</output_type>
-        <frame_name>laser_frame</frame_name>
-      </plugin>
+      </lidar>
     </sensor>
   </gazebo>

File: src/agv_sim_description/urdf/wheel_sim.xacro (robot description, xacro)
@@ -36,5 +36,4 @@
       <kp>1000000.0</kp>
       <kd>100.0</kd>
-      <material>Gazebo/Black</material>
     </gazebo>
   </xacro:macro>

Commit message: fix: ground plane position, ZED 2i visual, PBR textures, roof beams
- Ground plane: centered on greenhouse (pose 15,0,0), sized 34x19m
- ZED 2i: swapped box to 30x175x33mm (wide bar, not deep box), added
  lens cylinder indicators so camera clearly faces forward
- PBR materials: polycarbonate walls, dark foliage crops, galvanized
  steel rails, wooden crates, dirt ground, metallic chassis
- Greenhouse roof: 5 transverse + 2 longitudinal beams at Z=3.0m

File: src/agv_sim_description/urdf/agv_base_sim.xacro (robot description, xacro)
@@ -99,3 +99,13 @@
     <mu2>0.001</mu2>
   </gazebo>
+  <gazebo reference="base_link">
+    <visual>
+      <material>
+        <ambient>0.3 0.32 0.35 1</ambient>
+        <diffuse>0.4 0.42 0.45 1</diffuse>
+        <specular>0.3 0.3 0.3 1</specular>
+        <pbr><metal><metalness>0.4</metalness><roughness>0.5</roughness></metal></pbr>
+      </material>
+    </visual>
+  </gazebo>
 </robot>

File: src/agv_sim_description/urdf/sensors_sim.xacro (robot description, xacro)
@@ -8,5 +8,5 @@
     <visual>
       <geometry>
-        <box size="0.175 0.030 0.033"/>
+        <box size="0.030 0.175 0.033"/>
       </geometry>
       <material name="zed_dark_grey">
@@ -16,5 +16,5 @@
     <collision>
       <geometry>
-        <box size="0.175 0.030 0.033"/>
+        <box size="0.030 0.175 0.033"/>
       </geometry>
     </collision>
@@ -23,4 +23,24 @@
       <inertia ixx="0.00005" ixy="0" ixz="0" iyy="0.00005" iyz="0" izz="0.00005"/>
     </inertial>
+    <!-- Left lens indicator -->
+    <visual name="left_lens">
+      <origin xyz="0.016 0.06 0.0" rpy="0 1.5708 0"/>
+      <geometry>
+        <cylinder radius="0.008" length="0.003"/>
+      </geometry>
+      <material name="zed_lens">
+        <color rgba="0.1 0.1 0.15 1.0"/>
+      </material>
+    </visual>
+    <!-- Right lens indicator -->
+    <visual name="right_lens">
+      <origin xyz="0.016 -0.06 0.0" rpy="0 1.5708 0"/>
+      <geometry>
+        <cylinder radius="0.008" length="0.003"/>
+      </geometry>
+      <material name="zed_lens">
+        <color rgba="0.1 0.1 0.15 1.0"/>
+      </material>
+    </visual>
   </link>
   <joint name="zed_camera_joint" type="fixed">
