Commit message: fix: add PBR materials to all robot visual components
Wheels, casters, ZED camera body, and lidar frame now have proper
Gazebo PBR material overrides (ambient/diffuse/specular/metalness/
roughness). Previously these used only basic URDF colors which
ogre2 on NVIDIA cannot render through the fixed-function pipeline.

All world objects (walls, crops, rails, tags, ground) already had
PBR materials. This commit completes the robot body.

Note: 60 ogre2 material errors remain — these are gz-rendering
internal materials (scene::Material auto-IDs, Default/TransGreen,
highlight_material) incompatible with NVIDIA GL3Plus strict mode.
These are upstream gz-rendering bugs, not our scene materials.

Co-Authored-By: Claude Opus 4.6 (1M context) <noreply@anthropic.com>

File: src/agv_sim_description/urdf/agv_base_sim.xacro (robot description, xacro)
@@ -94,8 +94,24 @@
     <mu1>0.001</mu1>
     <mu2>0.001</mu2>
+    <visual>
+      <material>
+        <ambient>0.2 0.2 0.2 1</ambient>
+        <diffuse>0.3 0.3 0.3 1</diffuse>
+        <specular>0.15 0.15 0.15 1</specular>
+        <pbr><metal><metalness>0.3</metalness><roughness>0.6</roughness></metal></pbr>
+      </material>
+    </visual>
   </gazebo>
   <gazebo reference="rear_caster">
     <mu1>0.001</mu1>
     <mu2>0.001</mu2>
+    <visual>
+      <material>
+        <ambient>0.2 0.2 0.2 1</ambient>
+        <diffuse>0.3 0.3 0.3 1</diffuse>
+        <specular>0.15 0.15 0.15 1</specular>
+        <pbr><metal><metalness>0.3</metalness><roughness>0.6</roughness></metal></pbr>
+      </material>
+    </visual>
   </gazebo>
   <gazebo reference="base_link">

File: src/agv_sim_description/urdf/sensors_sim.xacro (robot description, xacro)
@@ -49,4 +49,14 @@
     <origin xyz="0.7 0.0 -0.055" rpy="0 0 0"/>
   </joint>
+  <gazebo reference="zed_camera_link">
+    <visual>
+      <material>
+        <ambient>0.12 0.12 0.12 1</ambient>
+        <diffuse>0.2 0.2 0.2 1</diffuse>
+        <specular>0.3 0.3 0.3 1</specular>
+        <pbr><metal><metalness>0.2</metalness><roughness>0.4</roughness></metal></pbr>
+      </material>
+    </visual>
+  </gazebo>
   <!-- Optical center between lenses (identity transform from camera body) -->
   <link name="zed_camera_center">
@@ -238,4 +248,12 @@
   </joint>
   <gazebo reference="laser_frame">
+    <visual>
+      <material>
+        <ambient>0.6 0.0 0.0 1</ambient>
+        <diffuse>0.8 0.0 0.0 1</diffuse>
+        <specular>0.3 0.1 0.1 1</specular>
+        <pbr><metal><metalness>0.1</metalness><roughness>0.5</roughness></metal></pbr>
+      </material>
+    </visual>
     <sensor name="lidar_sensor" type="gpu_lidar">
       <always_on>true</always_on>

File: src/agv_sim_description/urdf/wheel_sim.xacro (robot description, xacro)
@@ -36,4 +36,12 @@
       <kp>1000000.0</kp>
       <kd>100.0</kd>
+      <visual>
+        <material>
+          <ambient>0.05 0.05 0.05 1</ambient>
+          <diffuse>0.1 0.1 0.1 1</diffuse>
+          <specular>0.2 0.2 0.2 1</specular>
+          <pbr><metal><metalness>0.0</metalness><roughness>0.9</roughness></metal></pbr>
+        </material>
+      </visual>
     </gazebo>
   </xacro:macro>
