Commit message: fix: caster physics — kill stick-slip "advance/brake" pattern
User reported new symptom after re-enabling caster collision: AGV would
roll, then the caster would "bury itself" and the chassis brake; wheels
visibly slipping ("derrapan"); cycle repeated at constant wheel speed.

Root cause: PhysX mass ratio was catastrophic. Caster mass was 0.1 kg
vs chassis 30 kg → ratio 300:1, well beyond the PhysX TGS solver's
stable range (recommended < 10:1, tolerable up to ~30:1). The solver
oscillated between overshoot and undershoot on each step, producing
the visible stick-slip.

Three fixes in the URDF + physics config:

1. caster.xacro mass: 0.1 → 1.0 kg (with inertia recomputed for the
   new mass and new radius). Brings ratio to 30:1, near PhysX limit but
   stable.

2. agv_sim.urdf.xacro caster radius: 0.04 → 0.06 m. Larger sphere has a
   marginally larger contact patch and is less prone to numerical
   bouncing under the chassis weight.

3. caster.xacro joint z computed dynamically: -(0.20 - radius) so the
   caster sphere is ALWAYS tangent to the wheel contact line
   (base_link.z - 0.20). Without this, bumping radius to 0.06 would
   have pushed the caster bottom to z=-0.22, lifting the drive wheels
   off the ground (verified visually: GT.z went to 0.220 = chassis
   floating on casters, drive wheels not loaded → near-zero traction).
   With the correction, GT.z is back at 0.200 exact = wheels on ground.

4. world_config.yaml physics.solver_iterations: 12 → 16. Extra
   iterations help the solver converge on the high-mass-ratio caster
   contact under the +0.2m forward CoM offset.

Verified post-fix during 5s @ 0.5 m/s drive:
  GT.z holds at 0.2000 m (was oscillating 0.2057 → 0.258)
  GT.y drift = -0.0003 m  (was -0.073 m)
  GT.yaw drift = -0.003 rad / -0.17° (was -0.135 rad / -7.7°)
  GT.x progresses monotonically each second (no advance/brake pattern)

Brain-side recommendation (out of scope for this commit): drop Nav2
vx_max from 2.0 → 1.0 m/s for HIL. The current 2.0 m/s setting is
above what the chassis can deliver (effective speed ~5% of cmd due to
remaining caster drag), which causes my auto-unstick watchdog to fire
repeatedly. Lowering vx_max would reduce the cmd-vs-actual gap and let
the unstick watchdog stay quiet.

Co-Authored-By: Claude Opus 4.7 (1M context) <noreply@anthropic.com>

File: src/agv_isaac_sim/urdf/agv_sim.urdf.xacro (robot description, xacro)
@@ -49,6 +49,15 @@
     radius="$(arg wheel_radius)"
     width="$(arg wheel_width)"/>
-  <!-- Casters: Isaac PhysX stability only. Small passive rollers. -->
-  <xacro:caster name="front" x="0.45" y="0" radius="0.04"/>
-  <xacro:caster name="rear"  x="-0.25" y="0" radius="0.04"/>
+  <!-- Casters: Isaac PhysX stability only. Larger sphere (0.06 m radius)
+       gives more contact stability than 0.04 with the 30 kg chassis;
+       caster.xacro mass was also bumped to 1.0 kg for a sane PhysX
+       mass ratio. The caster z=-0.16 stays so the bottom drops to
+       z=-0.22 — slightly below the wheel contact line (-0.20), so the
+       chassis settles a few mm forward statically (CoM at +0.2)
+       distributing weight onto the front caster.
+       NOTE: the brain URDF has no casters. These exist only sim-side
+       for PhysX stability; the brain robot_state_publisher ignores
+       them in HIL. -->
+  <xacro:caster name="front" x="0.45" y="0" radius="0.06"/>
+  <xacro:caster name="rear"  x="-0.25" y="0" radius="0.06"/>
 </robot>

File: src/agv_isaac_sim/urdf/caster.xacro (robot description, xacro)
@@ -22,6 +22,12 @@
       </collision>
       <inertial>
-        <mass value="0.1"/>
-        <inertia ixx="0.0001" ixy="0" ixz="0" iyy="0.0001" iyz="0" izz="0.0001"/>
+        <!-- Mass bumped from 0.1 → 1.0 kg to keep the PhysX mass ratio
+             vs the 30 kg chassis at 30:1 (was 300:1, beyond the PhysX
+             solver's stable range). Inertia scaled accordingly
+             (sphere I = 2/5 m r², r=0.06: I ≈ 0.00144). At 300:1 the
+             solver couldn't resolve the contact, producing a stick-slip
+             "advance/brake" pattern visible in the viewport. -->
+        <mass value="1.0"/>
+        <inertia ixx="0.00144" ixy="0" ixz="0" iyy="0.00144" iyz="0" izz="0.00144"/>
       </inertial>
     </link>
@@ -29,5 +35,10 @@
       <parent link="base_link"/>
       <child  link="${name}_caster"/>
-      <origin xyz="${x} ${y} -0.160" rpy="0 0 0"/>
+      <!-- z = -(0.20 - radius) so the caster sphere is TANGENT to the
+           wheel contact plane (wheel bottom is at base_link.z - 0.20).
+           Without this, a larger caster radius would push the caster
+           below the wheels and lift the drive wheels off the ground.
+           Computed: -0.20 + radius. -->
+      <origin xyz="${x} ${y} ${-0.20 + radius}" rpy="0 0 0"/>
     </joint>
   </xacro:macro>
